Commit message: Added peg model and realtime visualization launcher.

File: kuka_lwr_description/robots/kuka_lwr_peg.xacro (robot description, xacro)
@@ -7,46 +7,32 @@
           <origin xyz="0.2 0.2 0" rpy="0 0 1.5708"/>
         </kuka_lwr_arm>
-	<!--joint name="target_frame" type="fixed">
-	  <origin xyz="0 0 0.235" rpy="1.5708 0 1.5708" />
-	  <parent link="right_arm_flange_link" />
-	  <child link="target_frame_link" />
-	</joint>
-	  <link name="target_frame_link">
-	    <inertial>
-	    <mass value="0.001" />
-	    <origin xyz="0 0 0" />
-	    <inertia ixx="0.0001" ixy="0.0" ixz="0.0"
-		    iyy="0.0001" iyz="0.0"
-		    izz="0.0001" />
-	  </inertial>
-	</link-->
-	<!--
-	<joint name="target_frame" type="fixed">
-	  <origin xyz="0 0 0.05" rpy="0 1.57 0" />
-	  <parent link="right_arm_flange_link" />
-	  <child link="dummy_link" />
-	</joint>
-	<link name="dummy_link">
-		<origin xyz="0 0 0" rpy="0 0 0"/>
-	</link>
-	<joint name="target_frame_two" type="fixed">
-	  <origin xyz="0 0 0" rpy="0 0 3.14" />
-	  <parent link="dummy_link" />
-	  <child link="peg_link" />
-	</joint>
-	<link name="peg_link">
-		<visual>
-			<origin xyz="0 0 0" rpy="0 0 0"/>
-			<geometry>
-   				<mesh filename="package://kuka_lwr_bringup/models/peg/peg.dae"/>
-			</geometry>
-        		</visual>
-		<collision>
-			<origin xyz="0 0 0" rpy="0 0 0"/>
-			<geometry>
-   				<mesh filename="package://kuka_lwr_bringup/models/peg/peg.dae"/>
-			</geometry>
-  		</collision>
-	</link>
--->
+     <joint name="target_frame" type="fixed">
+       <origin xyz="0 0 0.2" rpy="0 1.57 0" />
+       <parent link="right_arm_flange_link" />
+       <child link="dummy_link" />
+     </joint>
+     <link name="dummy_link">
+         <origin xyz="0 0 0" rpy="0 0 0"/>
+     </link>
+     <joint name="target_frame_two" type="fixed">
+       <origin xyz="0 0 0" rpy="0 0 3.14" />
+       <parent link="dummy_link" />
+       <child link="peg_link" />
+     </joint>
+     <link name="peg_link">
+         <visual>
+             <origin xyz="0 0 0" rpy="0 0 0"/>
+             <geometry>
+                    <mesh
+filename="package://kuka_lwr_bringup/models/peg/peg.dae"/>
+             </geometry>
+                 </visual>
+         <collision>
+             <origin xyz="0 0 0" rpy="0 0 0"/>
+             <geometry>
+                    <mesh
+filename="package://kuka_lwr_bringup/models/peg/peg.dae"/>
+             </geometry>
+           </collision>
+     </link>
 </robot>
