Commit message: Modified launch/urdf files for lwr2 setting.

File: kuka_lwr_description/robots/kuka_lwr2_lasa.urdf.xacro (robot description, xacro)
@@ -8,6 +8,9 @@
 	<xacro:include filename="$(find kuka_lwr_description)/urdf/kuka_lwr_arm_lasa.urdf.xacro"/>
 	<kuka_lwr_arm parent="leg4_link" name="right">
+          <origin xyz="1.39 0.15 0" rpy=" 0 0 1.6523"/>
+        </kuka_lwr_arm>
+	<!--kuka_lwr_arm parent="leg4_link" name="right">
           <origin xyz="1.39 0.15 0" rpy=" 0 0 3.141592"/>
-        </kuka_lwr_arm>
+        </kuka_lwr_arm -->
 	<joint name="op_table_top_joint" type="fixed" >
 	    <parent link="table_top_link" />

Commit message: Added plugin for visualization in Gazebo from Nicolas <3.

File: kuka_lwr_description/robots/kuka_lwr2_lasa.urdf.xacro (robot description, xacro)
@@ -28,17 +28,8 @@
 	    <child link="pole2_base_link" />
 	</joint>
-<!--	<joint name="target_frame" type="fixed">
-	  <origin xyz="0 0 0.235" rpy="1.5708 0 1.5708" />
-	  <parent link="right_arm_frame_link" />
-	  <child link="target_frame_link" />
-	</joint>
-	  <link name="target_frame_link">
-	    <inertial>
-	    <mass value="0.001" />
-	    <origin xyz="0 0 0" />
-	    <inertia ixx="0.0001" ixy="0.0" ixz="0.0"
-		    iyy="0.0001" iyz="0.0"
-		    izz="0.0001" />
-	  </inertial>
-	</link>-->
+    <gazebo>
+        <plugin name="set_joint_position" filename="libset_joint_position_plugin.so">
+            <topicName> /joint_states </topicName>
+        </plugin>
+    </gazebo>
 </robot>
