Commit message: modifications new/final setting

File: kuka_lwr_description/robots/kuka_bimanual2_lwr_lasa.urdf.xacro (robot description, xacro)
@@ -12,5 +12,5 @@
 	<xacro:include filename="$(find kuka_lwr_bringup)/models/table/table3b.urdf.xacro" />
 	<robot_dep_table parent="right_table_top_link" name="left">
-      <origin xyz="1.07 0 0" rpy=" 0 0 0"/>
+      <origin xyz="1.15 0 0" rpy=" 0 0 0"/>
     </robot_dep_table>
 	<xacro:include filename="$(find kuka_lwr_description)/urdf/kuka_lwr_arm_lasa.urdf.xacro"/>

Commit message: Slight changes to comply with bimanual simulation

File: kuka_lwr_description/robots/kuka_bimanual2_lwr_lasa.urdf.xacro (robot description, xacro)
@@ -8,5 +8,5 @@
 	<xacro:include filename="$(find kuka_lwr_description)/urdf/kuka_lwr_arm_lasa.urdf.xacro"/>
 	<kuka_lwr_arm parent="right_leg4_link" name="right">
-          <origin xyz="0.45 0.45 0" rpy=" 0 0 1.66"/>
+          <origin xyz="0.45 0.45 0" rpy=" 0 0 1.56"/>
         </kuka_lwr_arm>
 	<xacro:include filename="$(find kuka_lwr_bringup)/models/table/table3b.urdf.xacro" />
@@ -16,5 +16,5 @@
 	<xacro:include filename="$(find kuka_lwr_description)/urdf/kuka_lwr_arm_lasa.urdf.xacro"/>
 	<kuka_lwr_arm parent="left_leg4_link" name="left">
-          <origin xyz="0.45 0.39 0" rpy=" 0 0 1.7"/>
+          <origin xyz="0.45 0.39 0" rpy=" 0 0 1.56"/>
         </kuka_lwr_arm>
 	<xacro:include filename="$(find kuka_lwr_bringup)/models/pole/pole_kinect_table.urdf.xacro" />

Commit message: changed urdf and start configs in simulation for bimanual setting

File: kuka_lwr_description/robots/kuka_bimanual2_lwr_lasa.urdf.xacro (robot description, xacro)
@@ -16,5 +16,5 @@
 	<xacro:include filename="$(find kuka_lwr_description)/urdf/kuka_lwr_arm_lasa.urdf.xacro"/>
 	<kuka_lwr_arm parent="left_leg4_link" name="left">
-          <origin xyz="0.45 0.38 0" rpy=" 0 0 1.7"/>
+          <origin xyz="0.45 0.38 0" rpy=" 0 0 1.56"/>
         </kuka_lwr_arm>
 	<xacro:include filename="$(find kuka_lwr_bringup)/models/pole/pole_kinect_table.urdf.xacro" />
