Commit message: bimanual mods

File: kuka_lwr_description/robots/kuka_bimanual_lwr_lasa.urdf.xacro (robot description, xacro)
@@ -5,9 +5,13 @@
 	<xacro:include filename="$(find kuka_lwr_description)/urdf/kuka_lwr_arm_lasa.urdf.xacro"/>
 	<kuka_lwr_arm parent="leg4_link" name="left">
-          <origin xyz="1.4 0.15 0" rpy=" 0 0 3.141592"/>
+          <origin xyz="1.4 0.15 0" rpy=" 0 0 1.56"/>
         </kuka_lwr_arm>
 	<xacro:include filename="$(find kuka_lwr_description)/urdf/kuka_lwr_arm_lasa.urdf.xacro"/>
 	<kuka_lwr_arm parent="leg4_link" name="right">
-          <origin xyz="0.2 0.15 0" rpy=" 0 0 3.141592"/>
+          <origin xyz="0.2 0.15 0" rpy=" 0 0 1.56"/>
         </kuka_lwr_arm>
+	<!-- <xacro:include filename="$(find kuka_lwr_bringup)/models/Object/Object.urdf.xacro" />
+	<Object parent="leg4_link">
+          <origin xyz="0.6 -5.0 0" rpy=" 0 0 1.56"/>
+        </Object> -->
 </robot>

Commit message: Changed names for multi-robot setting.. cleaned up repo.. all working with 2 robots

File: kuka_lwr_description/robots/kuka_bimanual_lwr_lasa.urdf.xacro (robot description, xacro)
@@ -4,10 +4,10 @@
 	<xacro:include filename="$(find kuka_lwr_description)/defs/materials.xml"/>
 	<xacro:include filename="$(find kuka_lwr_description)/urdf/kuka_lwr_arm_lasa.urdf.xacro"/>
-	<kuka_lwr_arm parent="leg2_link" name="left">
-          <origin xyz="-0.0284889 -1.32351 0.105877" rpy=" 0 0 0"/>
+	<kuka_lwr_arm parent="leg2_link" name="first">
+          <origin xyz="0.20 -0.45 0.0" rpy=" 0 0 1.56"/>
         </kuka_lwr_arm>
 	<xacro:include filename="$(find kuka_lwr_description)/urdf/kuka_lwr_arm_lasa.urdf.xacro"/>
-	<kuka_lwr_arm parent="leg2_link" name="right">
-          <origin xyz="0.0 0.0 0" rpy=" 0 0 0"/>
+	<kuka_lwr_arm parent="leg2_link" name="second">
+          <origin xyz="1.40 -0.45 0" rpy=" 0 0 1.56"/>
         </kuka_lwr_arm>
 </robot>

Commit message: Multi-arm simulation working

File: kuka_lwr_description/robots/kuka_bimanual_lwr_lasa.urdf.xacro (robot description, xacro)
@@ -1,12 +1,15 @@
 <?xml version="1.0"?>
 <robot xmlns:xacro="http://www.ros.org/wiki/xacro" name="kuka_bimanual_lwr_description">
+	<xacro:include filename="$(find kuka_lwr_description)/defs/materials.xml"/>
 	<xacro:include filename="$(find kuka_lwr_bringup)/models/table/table2.urdf.xacro" />
-	<xacro:include filename="$(find kuka_lwr_description)/defs/materials.xml"/>
+	<robot_table name="one">
+      <origin xyz="0 0 0" rpy=" 0 0 0"/>
+    </robot_table>
 	<xacro:include filename="$(find kuka_lwr_description)/urdf/kuka_lwr_arm_lasa.urdf.xacro"/>
-	<kuka_lwr_arm parent="leg2_link" name="first">
+	<kuka_lwr_arm parent="one_leg2_link" name="first">
           <origin xyz="0.20 -0.45 0.0" rpy=" 0 0 1.56"/>
         </kuka_lwr_arm>
 	<xacro:include filename="$(find kuka_lwr_description)/urdf/kuka_lwr_arm_lasa.urdf.xacro"/>
-	<kuka_lwr_arm parent="leg2_link" name="second">
+	<kuka_lwr_arm parent="one_leg2_link" name="second">
           <origin xyz="1.40 -0.45 0" rpy=" 0 0 1.56"/>
         </kuka_lwr_arm>
