Commit message: Changed xacro files, removed annoying debug msgs from plugin.

File: kuka_lwr_bringup/models/pole/pole.urdf.xacro (robot description, xacro)
@@ -22,5 +22,5 @@
   <property name="pole_base_thickness" value="0.05"/>
   <property name="pole_base_color" value="0 0 0 1" />
-  <property name="pole_color" value="100 100 100 1" />
+  <property name="pole_color" value="0 0 0 1" />
   <property name="M_PI" value="3.1415926535897931" />
   <link name="pole_base_link">

File: kuka_lwr_bringup/models/pole/pole_2.urdf.xacro (robot description, xacro)
@@ -21,5 +21,5 @@
   <property name="pole2_z"      value="0.0" />
   <property name="pole2_base_color" value="0 0 0 1" />
-  <property name="pole2_color" value="100 100 100 1" />
+  <property name="pole2_color" value="0 0 0 1" />
   <property name="pole2_base_thickness" value="0.05"/>
   <property name="M_PI" value="3.1415926535897931" />

File: kuka_lwr_bringup/models/table/operation_table.urdf.xacro (robot description, xacro)
@@ -21,5 +21,5 @@
   <property name="op_table_z"      value="0.0" />
   <property name="op_table_top_thickness" value="0.025"/>
-  <property name="op_table_top_color" value="100 100 100 1" />
+  <property name="op_table_top_color" value="0 0 0 1" />
   <property name="op_leg_color" value="0 0 0 1" />
   <property name="M_PI" value="3.1415926535897931" />

File: kuka_lwr_description/robots/kuka_lwr2_lasa.urdf.xacro (robot description, xacro)
@@ -10,7 +10,4 @@
           <origin xyz="1.39 0.15 0" rpy=" 0 0 1.6523"/>
         </kuka_lwr_arm>
-	<!--kuka_lwr_arm parent="leg4_link" name="right">
-          <origin xyz="1.39 0.15 0" rpy=" 0 0 3.141592"/>
-        </kuka_lwr_arm -->
 	<joint name="op_table_top_joint" type="fixed" >
 	    <parent link="table_top_link" />
