Commit message: Added realtime visualization of bimanual setting + Kinect + Ft sensors!!

File: kuka_lwr_bringup/models/pole/pole_kinect_table.urdf.xacro (robot description, xacro)
@@ -180,5 +180,5 @@
     </inertial>
     <visual>
-      <origin xyz="0.0 -0.75 0.76" rpy="0 0 0" />
+      <origin xyz="0.0 -0.75 0.74" rpy="0 0 0" />
       <geometry>
         <box size="0.75 0.56 0.03" />
@@ -189,5 +189,5 @@
     </visual>
     <collision>
-      <origin xyz="0.0 -0.75 0.77" rpy="0 0 0" />
+      <origin xyz="0.0 -0.75 0.74" rpy="0 0 0" />
       <geometry>
         <box size="0.75 0.56 0.02" />

Commit message: Calibration for new bimanual setting

File: kuka_lwr_bringup/models/pole/pole_kinect_table.urdf.xacro (robot description, xacro)
@@ -180,5 +180,5 @@
     </inertial>
     <visual>
-      <origin xyz="0.0 -0.75 0.74" rpy="0 0 0" />
+      <origin xyz="0.0 -0.62 0.74" rpy="0 0 0" />
       <geometry>
         <box size="0.75 0.56 0.03" />
@@ -189,5 +189,5 @@
     </visual>
     <collision>
-      <origin xyz="0.0 -0.75 0.74" rpy="0 0 0" />
+      <origin xyz="0.0 -0.62 0.74" rpy="0 0 0" />
       <geometry>
         <box size="0.75 0.56 0.02" />

File: kuka_lwr_description/robots/kuka_bimanual2_lwr_lasa.urdf.xacro (robot description, xacro)
@@ -8,18 +8,18 @@
 	<xacro:include filename="$(find kuka_lwr_description)/urdf/kuka_lwr_arm_lasa.urdf.xacro"/>
 	<kuka_lwr_arm parent="right_leg4_link" name="right">
-          <origin xyz="0.45 0.45 0" rpy=" 0 0 1.56"/>
+          <origin xyz="0.45 0.45 0" rpy=" 0 0 1.66"/>
         </kuka_lwr_arm>
 	<xacro:include filename="$(find kuka_lwr_bringup)/models/table/table3b.urdf.xacro" />
 	<robot_dep_table parent="right_table_top_link" name="left">
-      <origin xyz="1.15 0 0" rpy=" 0 0 0"/>
+      <origin xyz="1.18 0 0" rpy=" 0 0 0"/>
     </robot_dep_table>
 	<xacro:include filename="$(find kuka_lwr_description)/urdf/kuka_lwr_arm_lasa.urdf.xacro"/>
 	<kuka_lwr_arm parent="left_leg4_link" name="left">
-          <origin xyz="0.45 0.38 0" rpy=" 0 0 1.56"/>
+          <origin xyz="0.45 0.39 0" rpy=" 0 0 1.7"/>
         </kuka_lwr_arm>
 	<xacro:include filename="$(find kuka_lwr_bringup)/models/pole/pole_kinect_table.urdf.xacro" />
 	<joint name="pole2_base_joint" type="fixed" >
 	    <parent link="right_table_top_link" />
-	    <origin xyz="0.53 0.25 ${pole2_base_thickness/2}" rpy="0 0 0" />
+	    <origin xyz="0.60 0.15 ${pole2_base_thickness/2}" rpy="0 0 0" />
 	    <child link="pole2_base_link" />
 	</joint>

Commit message: Recalibrated zucchini setting

File: kuka_lwr_bringup/models/pole/pole_kinect_table.urdf.xacro (robot description, xacro)
@@ -22,4 +22,5 @@
   <property name="pole2_base_color" value="0 0 0 1" />
   <property name="pole2_color" value="0 0 0 1" />
+  <property name="table_color" value="100 100 100 1" />
   <property name="pole2_base_thickness" value="0.05"/>
   <property name="M_PI" value="3.1415926535897931" />
@@ -180,15 +181,15 @@
     </inertial>
     <visual>
+      <origin xyz="0.02 -0.75 0.74" rpy="0 0 0" />
+      <geometry>
+        <box size="0.75 0.56 0.03" />
+      </geometry>
+      <material name="table_color">
+        <color rgba="100 100 100 1"/>
+      </material>
+    </visual>
+    <collision>
       <origin xyz="0.0 -0.75 0.74" rpy="0 0 0" />
       <geometry>
-        <box size="0.75 0.56 0.03" />
-      </geometry>
-      <material name="pole2_blue">
-        <color rgba="0 0 0 1"/>
-      </material>
-    </visual>
-    <collision>
-      <origin xyz="0.0 -0.75 0.74" rpy="0 0 0" />
-      <geometry>
         <box size="0.75 0.56 0.02" />
       </geometry>

File: kuka_lwr_description/robots/kuka_bimanual2_lwr_lasa.urdf.xacro (robot description, xacro)
@@ -12,14 +12,14 @@
 	<xacro:include filename="$(find kuka_lwr_bringup)/models/table/table3b.urdf.xacro" />
 	<robot_dep_table parent="right_table_top_link" name="left">
-      <origin xyz="1.15 0 0" rpy=" 0 0 0"/>
+      <origin xyz="1.15 0.05 0" rpy=" 0 0 0"/>
     </robot_dep_table>
 	<xacro:include filename="$(find kuka_lwr_description)/urdf/kuka_lwr_arm_lasa.urdf.xacro"/>
 	<kuka_lwr_arm parent="left_leg4_link" name="left">
-          <origin xyz="0.45 0.38 0" rpy=" 0 0 1.56"/>
+          <origin xyz="0.45 0.38 0" rpy=" 0 0 1.7"/>
         </kuka_lwr_arm>
 	<xacro:include filename="$(find kuka_lwr_bringup)/models/pole/pole_kinect_table.urdf.xacro" />
 	<joint name="pole2_base_joint" type="fixed" >
 	    <parent link="right_table_top_link" />
-	    <origin xyz="0.53 0.25 ${pole2_base_thickness/2}" rpy="0 0 0" />
+	    <origin xyz="0.53 0.25 ${pole2_base_thickness/2-0.02}" rpy="0 0 0" />
 	    <child link="pole2_base_link" />
 	</joint>
